File: NeuralCard.kicad_sch (KiCad schematic)
At the start: 53 parts, among them J1 ProgPads, SW1 SW_PUSH, SW2 SW_PUSH, U1 ESP32-S3-WROOM-1, U2 LSM6DS3TR-C, U4 ST25DV04KC-IE6S3

Commit message: fix(sch): add SW3 to the schematic so the board and netlist agree
SW3 was added straight to the layout in b2ccb56 and never had a schematic
symbol. The board carried a VBAT net with no schematic counterpart, so Update
PCB from Schematic would have flagged SW3 as an extra footprint and deleted
it, silently undoing the MSK12C02 DFM fix from a316055.

Fixed in gen_schematic.py rather than by hand-editing NeuralCard.kicad_sch,
so the switch survives the next regeneration. LIBSYMS gains Switch:SW_SPDT,
PIN_XY its pin geometry, FP maps SW3 to the MSK12C02 footprint, and
section_power() puts the switch in series between the coin and the rail:
BT1 pin 1 drives VBAT, SW3 pin 2 (common pole) takes VBAT, pin 3 (closed
throw) drives +3V3, pin 1 (open throw) gets an explicit no-connect.

KiCad's generic Switch:SW_SPDT numbers its common pole pin 2, matching the
MSK12C02 pinout and the pad nets already on the board, so the stock symbol is
used unmodified and no pin renumbering was needed.

Verification:

- The generator reproduces the previously committed schematic exactly (53
  nets, 53 components, 0 differences) before the switch is added, so
  regenerating loses nothing.
- Schematic netlist checked pad-by-pad against NeuralCard.kicad_pcb: 174
  schematic pads, 173 PCB pads, 0 net mismatches. The single difference is
  SW3 pad 1, unconnected on both sides. Update PCB from Schematic is now a
  connectivity no-op.
- ERC 0 errors, 41 warnings -- identical to the count before this change.

Also discards the uncommitted KiCad 10 re-save that was sitting in the working
tree (format 20250114->20260306, A2->A3); the schematic is back to the
generator's canonical KiCad 9 / A2 output.

Corrects DESIGN.md's stale "56 components / 56 warnings" to the verified 54
and 41, and records the 54-vs-52 schematic/CPL delta as ANT1 and J1.

No PCB, gerber, drill, BOM or CPL output is modified.
Parts:
- added SW3: MSK12C02, Button_Switch_SMD:SW_SPDT_Shouhan_MSK12C02, symbol Switch:SW_SPDT
Connections:
- net +3V3: now also SW3.3 (C); no longer BT1.1
- new net VBAT: BT1.1, SW3.2 (B)
- no-connect marks 29 -> 30
Other:
- note added: "POWER (CR2032 coin -> SW3 -> 3V3 rail; also fed by prog-pad 3V3)"
- note removed: "POWER (CR2032 coin -> 3V3 rail; also fed by prog-pad 3V3)"
Changed lines of the file:
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@@
 		)
 	)
-	(text "POWER  (CR2032 coin -> 3V3 rail; also fed by prog-pad 3V3)"
+	(text "POWER  (CR2032 coin -> SW3 -> 3V3 rail; also fed by prog-pad 3V3)"
 		(exclude_from_sim no)
 		(at 28 28 0)
@@
 		)
 	)
-	(symbol
-		(lib_id "power:+3V3")
-		(at 50.8 71.12 0)
+	(global_label "VBAT"
+		(shape bidirectional)
+		(at 50.8 71.11999999999999 0)
+		(effects
+			(font
+				(size 1.27 1.27)
+			)
+			(justify left)
+		)
+		(property "Intersheetrefs" "${INTERSHEET_REFS}"
+			(at 50.8 71.11999999999999 0)
+			(effects
+				(font
+					(size 1.27 1.27)
+				)
+				(hide yes)
+			)
+		)
+	)
+	(wire
+		(pts
+			(xy 60.96 73.66) (xy 60.96 76.2)
+		)
+		(stroke
+			(width 0)
+			(type default)
+		)
+	)
+	(symbol
+		(lib_id "power:GND")
+		(at 60.96 76.2 0)
 		(unit 1)
 		(exclude_from_sim no)
@@
 		(dnp no)
 		(property "Reference" "#PWR001"
-			(at 50.8 71.11999999999999 0)
-			(effects
-				(font
-					(size 1.27 1.27)
-				)
-			)
-			(hide yes)
-		)
-		(property "Value" "+3V3"
-			(at 50.8 67.81799999999998 0)
+			(at 60.96 76.2 0)
+			(effects
+				(font
+					(size 1.27 1.27)
+				)
+			)
+			(hide yes)
+		)
+		(property "Value" "GND"
+			(at 60.96 79.50200000000001 0)
 			(effects
 				(font
@@
 		)
 		(property "Footprint" ""
-			(at 50.8 71.11999999999999 0)
+			(at 60.96 76.2 0)
 			(effects
 				(font
@@
 		)
 		(property "Datasheet" ""
-			(at 50.8 71.11999999999999 0)
+			(at 60.96 76.2 0)
 			(effects
 				(font
@@
 		)
 		(property "Description" ""
-			(at 50.8 71.11999999999999 0)
+			(at 60.96 76.2 0)
 			(effects
 				(font
@@
 		)
 	)
+	(symbol
+		(lib_id "Switch:SW_SPDT")
+		(at 76.2 60.96 0)
+		(unit 1)
+		(exclude_from_sim no)
+		(in_bom yes)
+		(on_board yes)
+		(dnp no)
+		(property "Reference" "SW3"
+			(at 78.74000000000001 59.69 0)
+			(effects
+				(font
+					(size 1.27 1.27)
+				)
+				(justify left)
+			)
+		)
+		(property "Value" "MSK12C02"
+			(at 78.74000000000001 62.230000000000004 0)
+			(effects
+				(font
+					(size 1.27 1.27)
+				)
+				(justify left)
+			)
+		)
+		(property "Footprint" "Button_Switch_SMD:SW_SPDT_Shouhan_MSK12C02"
+			(at 76.2 60.96 0)
+			(effects
+				(font
+					(size 1.27 1.27)
+				)
+			)
+			(hide yes)
+		)
+		(property "Datasheet" ""
+			(at 76.2 60.96 0)
+			(effects
+				(font
+					(size 1.27 1.27)
+				)
+			)
+			(hide yes)
+		)
+		(property "Description" ""
+			(at 76.2 60.96 0)
+			(effects
+				(font
+					(size 1.27 1.27)
+				)
+			)
+			(hide yes)
+		)
+		(pin "1"
+		)
+		(pin "2"
+		)
+		(pin "3"
+		)
+		(instances
+			(project "NeuralCard"
+				(path "/a1b2c3d4-0001-4000-8000-000000000001"
+					(reference "SW3")
+					(unit 1)
+				)
+			)
+		)
+	)
 	(wire
 		(pts
-			(xy 60.96 73.66) (xy 60.96 76.2)
+			(xy 71.12 60.96) (xy 68.58 60.96)
 		)
 		(stroke
@@
 		)
 	)
-	(symbol
-		(lib_id "power:GND")
-		(at 60.96 76.2 0)
+	(global_label "VBAT"
+		(shape bidirectional)
+		(at 68.58 60.96 0)
+		(effects
+			(font
+				(size 1.27 1.27)
+			)
+			(justify right)
+		)
+		(property "Intersheetrefs" "${INTERSHEET_REFS}"
+			(at 68.58 60.96 0)
+			(effects
+				(font
+					(size 1.27 1.27)
+				)
+				(hide yes)
+			)
+		)
+	)
+	(wire
+		(pts
+			(xy 81.28 63.5) (xy 86.36 63.5)
+		)
+		(stroke
+			(width 0)
+			(type default)
+		)
+	)
+	(symbol
+		(lib_id "power:+3V3")
+		(at 86.36 63.5 0)
 		(unit 1)
 		(exclude_from_sim no)
@@
 		(dnp no)
 		(property "Reference" "#PWR002"
-			(at 60.96 76.2 0)
-			(effects
-				(font
-					(size 1.27 1.27)
-				)
-			)
-			(hide yes)
-		)
-		(property "Value" "GND"
-			(at 60.96 79.50200000000001 0)
+			(at 86.36 63.5 0)
+			(effects
+				(font
+					(size 1.27 1.27)
+				)
+			)
+			(hide yes)
+		)
+		(property "Value" "+3V3"
+			(at 86.36 60.198 0)
 			(effects
 				(font
@@
 		)
 		(property "Footprint" ""
-			(at 60.96 76.2 0)
+			(at 86.36 63.5 0)
 			(effects
 				(font
@@
 		)
 		(property "Datasheet" ""
-			(at 60.96 76.2 0)
+			(at 86.36 63.5 0)
 			(effects
 				(font
@@
 		)
 		(property "Description" ""
-			(at 60.96 76.2 0)
+			(at 86.36 63.5 0)
 			(effects
 				(font
@@
 		)
 	)
-	(symbol
+	(no_connect
+		(at 81.28 58.42)
+	)
+	(symbol

Commit message: fix: led value flag
Two findings from the first kicad-happy run, both fixed in the generator so
they survive regeneration.

RS-001: VBAT has no declared source. Fallout from the SW3 symbol -- a plain
label carries no pin type, so strict checkers read the net as undriven. Adds a
PWR_FLAG on VBAT. KiCad's own ERC passed without it; this satisfies the
stricter check.

LED Value said "blue" while the footprint (LED-SMD_L1.6-W0.8-R-RD) and the fab
BOM (C2286) have always been red. Corrected to "red". Safe to change:
tools/export_fab.py documents the fab BOM as hand-maintained and not generated
from the schematic, so no fab output moves.

Verified: netlist unchanged on every real pin, 174 schematic pads vs 173 PCB
pads with 0 mismatches, ERC still 0 errors and 41 warnings. The analyzer now
reports LED D1 (red) [resistor_limited] and RS-001 is gone.
Parts:
- D1, D10, D11, D12, D13, D14, D15, D16, D17, D18, D19, D2, D20, D21, D22, D23, D24, D3, D4, D5, D6, D7, D8, D9: value blue -> red
Changed lines of the file:
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@@
 		)
 	)
+	(symbol
+		(lib_id "power:PWR_FLAG")
+		(at 49.53 44.45 0)
+		(unit 1)
+		(exclude_from_sim no)
+		(in_bom yes)
+		(on_board yes)
+		(dnp no)
+		(property "Reference" "#FLG03"
+			(at 49.53 41.910000000000004 0)
+			(effects
+				(font
+					(size 1.27 1.27)
+				)
+			)
+			(hide yes)
+		)
+		(property "Value" "PWR_FLAG"
+			(at 49.53 41.910000000000004 0)
+			(effects
+				(font
+					(size 1.27 1.27)
+				)
+			)
+		)
+		(property "Footprint" ""
+			(at 49.53 44.45 0)
+			(effects
+				(font
+					(size 1.27 1.27)
+				)
+			)
+			(hide yes)
+		)
+		(property "Datasheet" ""
+			(at 49.53 44.45 0)
+			(effects
+				(font
+					(size 1.27 1.27)
+				)
+			)
+			(hide yes)
+		)
+		(property "Description" ""
+			(at 49.53 44.45 0)
+			(effects
+				(font
+					(size 1.27 1.27)
+				)
+			)
+			(hide yes)
+		)
+		(pin "1"
+		)
+		(instances
+			(project "NeuralCard"
+				(path "/a1b2c3d4-0001-4000-8000-000000000001"
+					(reference "#FLG03")
+					(unit 1)
+				)
+			)
+		)
+	)
+	(wire
+		(pts
+			(xy 49.53 44.45) (xy 49.53 46.99)
+		)
+		(stroke
+			(width 0)
+			(type default)
+		)
+	)
+	(global_label "VBAT"
+		(shape bidirectional)
+		(at 49.53 46.99 0)
+		(effects
+			(font
+				(size 1.27 1.27)
+			)
+			(justify left)
+		)
+		(property "Intersheetrefs" "${INTERSHEET_REFS}"
+			(at 49.53 46.99 0)
+			(effects
+				(font
+					(size 1.27 1.27)
+				)
+				(hide yes)
+			)
+		)
+	)
 	(rectangle
 		(start 26 112)
@@
 			)
 		)
-		(property "Value" "blue"
+		(property "Value" "red"
 			(at 60.96 302.514 0)
 			(effects
@@
 			)
 		)
-		(property "Value" "blue"
+		(property "Value" "red"
 			(at 111.76 302.514 0)
 			(effects
@@
 			)
 		)
-		(property "Value" "blue"
+		(property "Value" "red"
 			(at 162.56 302.514 0)
 			(effects
@@
 			)
 		)
-		(property "Value" "blue"
+		(property "Value" "red"
 			(at 213.36 302.514 0)
 			(effects
@@
 			)
 		)
-		(property "Value" "blue"
+		(property "Value" "red"
 			(at 264.16 302.514 0)
 			(effects
@@
 			)
 		)
-		(property "Value" "blue"
+		(property "Value" "red"
 			(at 314.96 302.514 0)
 			(effects
@@
 			)
 		)
-		(property "Value" "blue"
+		(property "Value" "red"
 			(at 60.96 321.56399999999996 0)
 			(effects
@@
 			)
 		)
-		(property "Value" "blue"
+		(property "Value" "red"
 			(at 111.76 321.56399999999996 0)
 			(effects
@@
 			)
 		)
-		(property "Value" "blue"
+		(property "Value" "red"
 			(at 162.56 321.56399999999996 0)
 			(effects
@@
 			)
 		)
-		(property "Value" "blue"
+		(property "Value" "red"
 			(at 213.36 321.56399999999996 0)
 			(effects
@@
 			)
 		)
-		(property "Value" "blue"
+		(property "Value" "red"
 			(at 264.16 321.56399999999996 0)
 			(effects
@@
 			)
 		)
-		(property "Value" "blue"
+		(property "Value" "red"
 			(at 314.96 321.56399999999996 0)
 			(effects
@@
 			)
 		)
-		(property "Value" "blue"
+		(property "Value" "red"
 			(at 60.96 340.614 0)
 			(effects
@@
 			)
 		)
-		(property "Value" "blue"
+		(property "Value" "red"
 			(at 111.76 340.614 0)
 			(effects
@@
 			)
 		)
-		(property "Value" "blue"
+		(property "Value" "red"
 			(at 162.56 340.614 0)
 			(effects
@@
 			)
 		)
-		(property "Value" "blue"
+		(property "Value" "red"
 			(at 213.36 340.614 0)
 			(effects
@@
 			)
 		)
-		(property "Value" "blue"
+		(property "Value" "red"
 			(at 264.16 340.614 0)
 			(effects
@@
 			)
 		)
-		(property "Value" "blue"
+		(property "Value" "red"
 			(at 314.96 340.614 0)
 			(effects
@@
 			)
 		)
-		(property "Value" "blue"
+		(property "Value" "red"
 			(at 60.96 359.664 0)
 			(effects
@@
 			)
 		)
-		(property "Value" "blue"
+		(property "Value" "red"
 			(at 111.76 359.664 0)
 			(effects
@@
 			)
 		)
-		(property "Value" "blue"
+		(property "Value" "red"
 			(at 162.56 359.664 0)
 			(effects
@@
 			)
 		)
-		(property "Value" "blue"
+		(property "Value" "red"
 			(at 213.36 359.664 0)
 			(effects
@@
 			)
 		)
-		(property "Value" "blue"
+		(property "Value" "red"
 			(at 264.16 359.664 0)
 			(effects
@@
 			)
 		)
-		(property "Value" "blue"
+		(property "Value" "red"
 			(at 314.96 359.664 0)
 			(effects

Commit message: feat: add bom mpns
Part numbers now live in the schematic instead of only BOM_JLCPCB.csv. Adds
MPN, Manufacturer and LCSC properties on every purchasable component, plus
BOM Comments notes for the four parts with ordering caveats.

Canonical kicad-happy field names, since the project had no prior convention.
MPNs verified against the LCSC/jlcsearch API on 2026-08-02; manufacturer names
come from the LCSC catalogue, which the API does not expose.

Coverage is 15/18 BOM lines. The three without a part number are correct:
ANT1 and J1 are bare copper, and C12 is deliberately select-at-order pending a
VNA trim.

Clears SS-001 ("BOM has <50% MPN coverage, board is not pre-fab ready") and
enables the lifecycle audit, which now checks 14 parts instead of skipping.
Total findings 88 -> 86. ERC unchanged at 0 errors and 41 warnings.

This is the structural fix for the class of bug that let SW3 sit as
select-at-order until a fab rejected it.
Parts:
- BT1: LCSC (none) -> C70377; MPN (none) -> CR2032-BS-6-1; Manufacturer (none) -> Q&J
- C1, C11, C2, C3, C4, C5: LCSC (none) -> C14663; MPN (none) -> CC0603KRX7R9BB104; Manufacturer (none) -> YAGEO
- C10: BOM Comments (none) -> 22uF substitute -- no basic 100uF exists in 0805.; LCSC (none) -> C45783; MPN (none) -> CL21A226MAQNNNE; Manufacturer (none) -> Samsung Electro-Mechanics
- C12: BOM Comments (none) -> Select at order: any 0603 NP0/C0G, 56-68pF. Trim to 13.56MH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
- C8: LCSC (none) -> C15850; MPN (none) -> CL21A106KAYNNNE; Manufacturer (none) -> Samsung Electro-Mechanics
- C9: LCSC (none) -> C45783; MPN (none) -> CL21A226MAQNNNE; Manufacturer (none) -> Samsung Electro-Mechanics
- D1, D10, D11, D12, D13, D14, D15, D16, D17, D18, D19, D2, D20, D21, D22, D23, D24, D3, D4, D5, D6, D7, D8, D9: LCSC (none) -> C2286; MPN (none) -> KT-0603R; Manufacturer (none) -> Hubei KENTO Elec
- R1, R2, R3, R4, R5, R6: LCSC (none) -> C22962; MPN (none) -> 0603WAF2200T5E; Manufacturer (none) -> UNI-ROYAL
- R10, R9: LCSC (none) -> C25804; MPN (none) -> 0603WAF1002T5E; Manufacturer (none) -> UNI-ROYAL
- R11, R12: LCSC (none) -> C23162; MPN (none) -> 0603WAF4701T5E; Manufacturer (none) -> UNI-ROYAL
- R14: LCSC (none) -> C25803; MPN (none) -> 0603WAF1003T5E; Manufacturer (none) -> UNI-ROYAL
- SW1, SW2: LCSC (none) -> C318884; MPN (none) -> TS-1187A-B-A-B; Manufacturer (none) -> XKB Connection
- SW3: BOM Comments (none) -> Right-angle SPDT. Datasheet-exact land including 4 shield t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; LCSC (none) -> C431540; MPN (none) -> MSK12C02; Manufacturer (none) -> SHOU HAN
- U1: BOM Comments (none) -> N8R2, not N16R8. PSRAM pins are NC and the int8 model fits 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; LCSC (none) -> C2913204; MPN (none) -> ESP32-S3-WROOM-1-N8R2; Manufacturer (none) -> Espressif Systems
- U2: LCSC (none) -> C967633; MPN (none) -> LSM6DS3TR-C; Manufacturer (none) -> STMicroelectronics
- U4: LCSC (none) -> C3304276; MPN (none) -> ST25DV04KC-IE6S3; Manufacturer (none) -> STMicroelectronics
