File: hardware/NeuralCard.kicad_pcb (KiCad board)
At the start: 2 copper layers, 85.6 x 54 mm, 66 parts, among them J1 ProgPads, J2 TYPE-C-31-M-12, Q1 AO3401A, SW1 SW-SMD_4P-L5.1-W5.1-P3.70-LS6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, SW2 SW-SMD_4P-L5.1-W5.1-P3.70-LS6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, SW3 SW_SPDT_Shouhan_MSK12C02, U1 WIRELM-SMD_ESP32-S3-WROOM-1, U2 LGA-14_L3.0-W2.5-P0.50-TL, U3 ME6211C33M5G-N, U4 SO-8_L4.9-W3.9-P1.27-LS5.9-BL, U5 USBLC6-2SC6

Commit message: fixed contents
Parts:
- added C13: 4.7uF, C_0603_1608Metric, B.Cu at (48.0, 16.0)
- added C14: 4.7uF, C_0603_1608Metric, B.Cu at (52.0, 16.5)
- added D25: B5819W, D_SOD-123, B.Cu at (69.0, 10.5)
- added FID1: Fiducial_1mm_Mask2mm, Fiducial_1mm_Mask2mm, B.Cu at (3.50, 3.00)
- added R15: 20k, R_0603_1608Metric, B.Cu at (57.0, 11.5)
- added U6: MCP73831T-2ACI/OT, SOT-23-5_L3.0-W1.7-P0.95-LS2.8-BL, B.Cu at (52.0, 12.0)
- BT1: value BAT-TH_CR2032-BS-6-1 -> LIR2450; footprint BAT-TH_CR2032-BS-6-1 -> BatteryHolder_Keystone_3009_1x2450
- moved FID4 77.5 mm to (81.0, 3.00)
- moved R14 27.2 mm to (44.0, 31.5), turned to 90 degrees
- moved C10 2.60 mm to (77.4, 4.50)
- moved C7 0.30 mm to (79.0, 7.70)
- renumbered FID1 to FID4
Connections:
- C6 pad 1: VBUS -> VSYS
- Q1 pad 2: VBAT_SW -> VSYS
- Q1 pad 3: +3V3 -> VBAT_SW
- U3 pad 1: VBUS -> VSYS
- U3 pad 3: VBUS -> VSYS
- U3 pad 4: (no net) -> unconnected-(U3-NC-Pad4)
Routing:
- net GND: track 196.3 -> 508.0 mm, vias 50 -> 2
- net CP4: track 136.9 -> 224.9 mm
- net EN: track 108.9 -> 194.0 mm, vias 2 -> 0
- net CP3: track 155.7 -> 238.9 mm, vias 5 -> 3
- net CP2: track 178.2 -> 252.7 mm, vias 5 -> 1
- net VBAT: track 3.45 -> 53.9 mm
- net CP5: track 151.0 -> 201.2 mm, vias 8 -> 1
- net CP1: track 128.2 -> 164.3 mm, vias 3 -> 1
- net VSYS: track 0.00 -> 34.6 mm, vias 0 -> 2
- net NFC_GPO: track 100.5 -> 68.1 mm, vias 2 -> 4
- net VBUS: track 45.8 -> 67.1 mm, vias 6 -> 0
- net USB_DP: track 108.3 -> 87.4 mm, vias 12 -> 2
- net SDA: track 97.8 -> 78.8 mm, vias 3 -> 2
- net CP6: track 109.6 -> 124.4 mm
- net CHX3: track 28.7 -> 43.3 mm, vias 0 -> 2
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- removed copper zone on B.Cu, net GND
- removed copper zone on F.Cu, net GND
Other:
- board text added: "CR2032 ·"
- board text added: "NEURALCARD v3.0.0 2026"
- board text removed: "CR2032 · + side out"
- board text removed: "FLASH: hold BOOT · tap RST · release BOOT"
- board text removed: "NEURALCARD v2.3.1 · 2026"
- board text removed: "NeuralCard v2.3.1 · princetekki.com"
- board text removed: "OSHW · github.com/Brillar0101"

Commit message: correct switch pin mapping
Connections:
- SW1 pad 2: GND -> IO0
- SW1 pad 3: IO0 -> GND
- SW2 pad 1: EN -> GND
- SW2 pad 4: GND -> EN
Routing:
- net IO0: track 138.9 -> 141.2 mm
- net EN: track 194.0 -> 196.3 mm
Other:
- board text added: "NEURALCARD v3.0.1-dev"
- board text removed: "NEURALCARD v3.0.0 2026"
Changed lines of the file:
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@@
 		(title "NeuralCard")
 		(date "2026-08-07")
-		(rev "v3.0.0-dev")
+		(rev "v3.0.1-dev")
 	)
 	(layers
@@
 			(size 1 0.75)
 			(layers "B.Cu" "B.Mask" "B.Paste")
-			(net "GND")
+			(net "IO0")
 		)
 		(pad "3" smd rect
@@
 			(size 1 0.75)
 			(layers "B.Cu" "B.Mask" "B.Paste")
-			(net "IO0")
+			(net "GND")
 		)
 		(pad "4" smd rect
@@
 			(size 1 0.75)
 			(layers "B.Cu" "B.Mask" "B.Paste")
-			(net "EN")
+			(net "GND")
 		)
 		(pad "2" smd rect
@@
 			(size 1 0.75)
 			(layers "B.Cu" "B.Mask" "B.Paste")
-			(net "GND")
+			(net "EN")
 		)
 		(embedded_fonts no)
@@
 		)
 	)
-	(gr_text "NEURALCARD v3.0.0 2026"
+	(gr_text "NEURALCARD v3.0.1-dev"
 		(at 84.2 33 90)
 		(layer "F.SilkS")
@@
 	)
 	(segment
-		(start 15 49.15)
-		(end 15 46.0867)
-		(width 0.2)
-		(layer "B.Cu")
-		(net "GND")
-	)
-	(segment
 		(start 22.1033 36.025)
 		(end 22.1033 49.7867)
@@
 	)
 	(segment
-		(start 27 49.15)
-		(end 27 45.45)
-		(width 0.2)
-		(layer "B.Cu")
-		(net "GND")
-	)
-	(segment
 		(start 62 28)
 		(end 56.3 22.3)
@@
 	)
 	(segment
-		(start 27 49.7867)
-		(end 22.1033 49.7867)
+		(start 15 45.7683)
+		(end 18.3817 49.15)
 		(width 0.2)
 		(layer "B.Cu")
@@
 	)
 	(segment
-		(start 27 49.15)
-		(end 27 49.7867)
-		(width 0.2)
-		(layer "B.Cu")
-		(net "GND")
-	)
-	(segment
 		(start 52 10.85)
 		(end 52 11.5986)
@@
 	)
 	(segment
+		(start 18.3817 49.15)
+		(end 21 49.15)
+		(width 0.2)
+		(layer "B.Cu")
+		(net "GND")
+	)
+	(segment
 		(start 31.9 26.77)
 		(end 30.5 26.77)
@@
 	)
 	(segment
+		(start 22.1033 49.7867)
+		(end 21 49.15)
+		(width 0.2)
+		(layer "B.Cu")
+		(net "GND")
+	)
+	(segment
 		(start 26.275 8.844416)
 		(end 24.490584 7.06)
@@
 	)
 	(segment
+		(start 9 45.45)
+		(end 15 45.45)
+		(width 0.2)
+		(layer "B.Cu")
+		(net "GND")
+	)
+	(segment
 		(start 49.05 15.725)
 		(end 50.4874 15.725)
@@
 	)
 	(segment
-		(start 15 49.15)
-		(end 15 49.7867)
-		(width 0.2)
-		(layer "B.Cu")
-		(net "GND")
-	)
-	(segment
 		(start 73.8523 17)
 		(end 73.4639 17.3884)
@@
 	)
 	(segment
-		(start 15 45.7683)
-		(end 15 46.0867)
-		(width 0.2)
-		(layer "B.Cu")
-		(net "GND")
-	)
-	(segment
 		(start 34.199 6.1223)
 		(end 27.6721 12.6492)
@@
 	)
 	(segment
+		(start 21 49.15)
+		(end 27 49.15)
+		(width 0.2)
+		(layer "B.Cu")
+		(net "GND")
+	)
+	(segment
 		(start 44.7943 20.4307)
 		(end 44 21.225)
@@
 	)
 	(segment
-		(start 22.1033 49.7867)
-		(end 15 49.7867)
-		(width 0.2)
-		(layer "B.Cu")
-		(net "GND")
-	)
-	(segment
 		(start 67.5283 49.2669)
 		(end 67.5283 50)
@@
 	)
 	(segment
-		(start 21 49.15)
-		(end 21 45.45)
-		(width 0.2)
-		(layer "B.Cu")
-		(net "EN")
-	)
-	(segment
 		(start 82.240979 53.579853)
 		(end 82.24084 53.58)
@@
 	)
 	(segment
+		(start 21 45.45)
+		(end 27 45.45)
+		(width 0.2)
+		(layer "B.Cu")
+		(net "EN")
+	)
+	(segment
 		(start 64.3657 38.4586)
 		(end 57.2315 38.4586)
@@
 	)
 	(segment
-		(start 9 45.45)
-		(end 9 49.15)
+		(start 9 49.15)
+		(end 15 49.15)
 		(width 0.2)
 		(layer "B.Cu")
