File: hardware/NeuralCard.kicad_sch (KiCad schematic)
At the start: 63 parts, among them J1 ProgPads, J2 TYPE-C-31-M-12, Q1 AO3401A, SW1 SW_PUSH, SW2 SW_PUSH, SW3 MSK12C02, U1 ESP32-S3-WROOM-1, U2 LSM6DS3TR-C, U3 ME6211C33M5G-N, U4 ST25DV04KC-IE6S3, U5 USBLC6-2SC6

Commit message: fixed contents
Parts:
- removed BT1: CR2032, JLC:BAT-TH_CR2032-BS-6-1, symbol JLC:CR2032-BS-6-1
- removed J2: TYPE-C-31-M-12, JLC:USB-C_SMD-TYPE-C-31-M-12_1, symbol JLC:TYPE-C-31-M-12
- removed Q1: AO3401A, JLC:SOT-23_L2.9-W1.3-P1.90-LS2.4-BR, symbol JLC:AO3401A
- removed SW1, SW2: SW_PUSH, JLC:SW-SMD_4P-L5.1-W5.1-P3.70-LS6.5-TL_H1.5, symbol JLC:TS-1187A-B-A-B
- removed U1: ESP32-S3-WROOM-1, JLC:WIRELM-SMD_ESP32-S3-WROOM-1, symbol JLC:ESP32-S3-WROOM-1
- removed U2: LSM6DS3TR-C, JLC:LGA-14_L3.0-W2.5-P0.50-TL, symbol JLC:LSM6DS3TR-C
- removed U3: ME6211C33M5G-N, JLC:SOT-23-5_L3.0-W1.7-P0.95-LS2.8-BL, symbol JLC:ME6211C33M5G-N
- removed U5: USBLC6-2SC6, JLC:SOT-23-6_L2.9-W1.6-P0.95-LS2.8-BL, symbol JLC:USBLC6-2SC6
- added BT1: LIR2450, Battery:BatteryHolder_Keystone_3009_1x2450, symbol Parts:CR2032-BS-6-1
- added C13, C14: 4.7uF, Capacitor_SMD:C_0603_1608Metric, symbol Device:C
- added D25: B5819W, Diode_SMD:D_SOD-123, symbol Device:D_Schottky
- added J2: TYPE-C-31-M-12, Parts:USB-C_SMD-TYPE-C-31-M-12_1, symbol Parts:TYPE-C-31-M-12
- added Q1: AO3401A, Parts:SOT-23_L2.9-W1.3-P1.90-LS2.4-BR, symbol Parts:AO3401A
- added R15: 20k, Resistor_SMD:R_0603_1608Metric, symbol Device:R
- added SW1, SW2: SW_PUSH, Parts:SW-SMD_4P-L5.1-W5.1-P3.70-LS6.5-TL_H1.5, symbol Parts:TS-1187A-B-A-B
- added U1: ESP32-S3-WROOM-1, Parts:WIRELM-SMD_ESP32-S3-WROOM-1, symbol Parts:ESP32-S3-WROOM-1
- added U2: LSM6DS3TR-C, Parts:LGA-14_L3.0-W2.5-P0.50-TL, symbol Parts:LSM6DS3TR-C
- added U3: ME6211C33M5G-N, Parts:SOT-23-5_L3.0-W1.7-P0.95-LS2.8-BL, symbol Parts:ME6211C33M5G-N
- added U5: USBLC6-2SC6, Parts:SOT-23-6_L2.9-W1.6-P0.95-LS2.8-BL, symbol Parts:USBLC6-2SC6
- added U6: MCP73831T-2ACI/OT, Parts:SOT-23-5_L3.0-W1.7-P0.95-LS2.8-BL, symbol Battery_Management:MCP73831-2-OT
- C10: value 22uF -> 100uF
- D1, D10, D11, D12, D13, D14, D15, D16, D17, D18, D19, D2, D20, D21, D22, D23, D24, D3, D4, D5, D6, D7, D8, D9: footprint JLC:LED-SMD_L1.6-W0.8-R-RD -> Parts:LED-SMD_L1.6-W0.8-R-RD
Connections:
- net +3V3: now also U1.2 (3V3), U2.1 (SDO/SA0), U2.12 (CS), U2.5 (VDDIO), U2.8 (VDD), U3.5 (VOUT)
- net CC1: now also J2.A5 (CC1)
- net CC2: now also J2.B5 (CC2)
- net CHX1: now also U1.4 (IO4)
- net CHX2: now also U1.5 (IO5)
- net CHX3: now also U1.6 (IO6)
- net CHX4: now also U1.7 (IO7)
- net CHX5: now also U1.8 (IO15)
- net CHX6: now also U1.9 (IO16)
- net EN: now also SW2.1, SW2.3, U1.3 (EN)
- net GND: now also BT1.2, C13.2, C14.2, J2.1 (EH), J2.2 (EH), J2.3 (EH), J2.4 (EH), J2.A1B12 (GND), J2.B1A12 (GND), R15.2, SW1.2, SW1.4, SW2.2, SW2.4, U1.1 (GND), U1.40 (GND), U1.41 (GND), U2.6 (GND), U2.7 (GND), U3.2 (VSS), U5.2, U6.2 (V_{SS})
- net IMU_INT: now also U1.11 (IO18), U2.4 (INT1)
- net IO0: now also SW1.1, SW1.3, U1.27 (IO0)
- net NFC_GPO: now also U1.23 (IO21)
- net RXD: now also U1.36 (RXD0)
- net SCL: now also U1.10 (IO17), U2.13 (SCL)
- net SDA: now also U1.12 (IO8), U2.14 (SDA)
- net TXD: now also U1.37 (TXD0)
- net USB_DM: now also J2.A7 (DN1), J2.B7 (DN2), U1.13 (IO19), U5.3, U5.4
- net USB_DP: now also J2.A6 (DP1), J2.B6 (DP2), U1.14 (IO20), U5.1, U5.6
- net VBAT: now also BT1.1, C13.1, U6.3 (V_{BAT})
- net VBAT_SW: now also Q1.3 (D)
- net VBUS: now also C14.1, D25.2 (A), J2.A4B9 (VBUS), J2.B4A9 (VBUS), Q1.1 (G), U5.5, U6.4 (V_{DD}); no longer C6.1
- new net PROG: R15.1, U6.5 (PROG)
- new net VSYS: C6.1, D25.1 (K), Q1.2 (S), U3.1 (VIN), U3.3 (CE)
- no-connect marks 31 -> 32
Other:
- note added: "CHARGER (MCP73831: VBUS -> VBAT, 50mA)"
- note added: "POWER (LIR2450 coin -> SW3 -> VBAT_SW -> Q1 P-FET -> VSYS -> LDO)"
- note added: "USB-C (VBUS -> D25 -> VSYS -> ME6211 3.3V LDO; Q1 P-FET puts LIR2450 on VSYS when USB absent; USBLC6 ESD)"
- note removed: "POWER (CR2032 coin -> SW3 -> VBAT_SW -> Q1 P-FET -> 3V3 rail)"
- note removed: "USB-C (VBUS -> ME6211 3.3V LDO; Q1 P-FET isolates coin when USB present; USBLC6 ESD)"

Commit message: correct switch pin mapping
Connections:
- net EN: now also SW2.4; no longer SW2.1
- net GND: now also SW1.3, SW2.1; no longer SW1.2, SW2.4
- net IO0: now also SW1.2; no longer SW1.3
Changed lines of the file:
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@@
 	(title_block
 		(title "NeuralCard")
-		(rev "v3.0.0-dev")
+		(rev "v3.0.1-dev")
 		(company "Barakaeli Lawuo")
 		(comment 1 "AI business card - air-writing digit recognition, ESP32-S3")
@@
 		)
 	)
-	(global_label "EN"
+	(global_label "GND"
 		(shape bidirectional)
 		(at 55.88 147.32 0)
@@
 		)
 	)
-	(symbol
-		(lib_id "power:GND")
+	(global_label "EN"
+		(shape bidirectional)
 		(at 71.12 154.94 0)
-		(unit 1)
-		(exclude_from_sim no)
-		(in_bom yes)
-		(on_board yes)
-		(dnp no)
-		(property "Reference" "#PWR021"
-			(at 71.12 154.94 0)
-			(effects
-				(font
-					(size 1.27 1.27)
-				)
-			)
-			(hide yes)
-		)
-		(property "Value" "GND"
-			(at 71.12 158.242 0)
-			(effects
-				(font
-					(size 1.27 1.27)
-				)
-			)
-		)
-		(property "Footprint" ""
-			(at 71.12 154.94 0)
-			(effects
-				(font
-					(size 1.27 1.27)
-				)
-			)
-			(hide yes)
-		)
-		(property "Datasheet" ""
-			(at 71.12 154.94 0)
-			(effects
-				(font
-					(size 1.27 1.27)
-				)
-			)
-			(hide yes)
+		(effects
+			(font (size 1.27 1.27))
+			(justify left)
 		)
-		(property "Description" ""
+		(property "Intersheetrefs" "${INTERSHEET_REFS}"
 			(at 71.12 154.94 0)
-			(effects
-				(font
-					(size 1.27 1.27)
-				)
-			)
-			(hide yes)
-		)
-		(pin "1"
-		)
-		(instances
-			(project "NeuralCard"
-				(path "/a1b2c3d4-0001-4000-8000-000000000001"
-					(reference "#PWR021")
-					(unit 1)
-				)
-			)
+			(effects (font (size 1.27 1.27)) (hide yes))
 		)
 	)
@@
 		)
 	)
-	(global_label "IO0"
+	(global_label "GND"
 		(shape bidirectional)
 		(at 191.77 154.94 0)
@@
 		)
 	)
-	(symbol
-		(lib_id "power:GND")
+	(global_label "IO0"
+		(shape bidirectional)
 		(at 207.01 147.32 0)
-		(unit 1)
-		(exclude_from_sim no)
-		(in_bom yes)
-		(on_board yes)
-		(dnp no)
-		(property "Reference" "#PWR023"
-			(at 207.01 147.32 0)
-			(effects
-				(font
-					(size 1.27 1.27)
-				)
-			)
-			(hide yes)
-		)
-		(property "Value" "GND"
-			(at 207.01 150.62199999999999 0)
-			(effects
-				(font
-					(size 1.27 1.27)
-				)
-			)
-		)
-		(property "Footprint" ""
-			(at 207.01 147.32 0)
-			(effects
-				(font
-					(size 1.27 1.27)
-				)
-			)
-			(hide yes)
-		)
-		(property "Datasheet" ""
-			(at 207.01 147.32 0)
-			(effects
-				(font
-					(size 1.27 1.27)
-				)
-			)
-			(hide yes)
-		)
-		(property "Description" ""
+		(effects (font (size 1.27 1.27)) (justify left))
+		(property "Intersheetrefs" "${INTERSHEET_REFS}"
 			(at 207.01 147.32 0)
-			(effects
-				(font
-					(size 1.27 1.27)
-				)
-			)
-			(hide yes)
-		)
-		(pin "1"
-		)
-		(instances
-			(project "NeuralCard"
-				(path "/a1b2c3d4-0001-4000-8000-000000000001"
-					(reference "#PWR023")
-					(unit 1)
-				)
-			)
+			(effects (font (size 1.27 1.27)) (hide yes))
 		)
 	)
@@
 		)
 	)
-	(symbol
-		(lib_id "power:GND")
+	(global_label "GND"
+		(shape bidirectional)
 		(at 207.01 154.94 0)
-		(unit 1)
-		(exclude_from_sim no)
-		(in_bom yes)
-		(on_board yes)
-		(dnp no)
-		(property "Reference" "#PWR024"
-			(at 207.01 154.94 0)
-			(effects
-				(font
-					(size 1.27 1.27)
-				)
-			)
-			(hide yes)
-		)
-		(property "Value" "GND"
-			(at 207.01 158.242 0)
-			(effects
-				(font
-					(size 1.27 1.27)
-				)
-			)
-		)
-		(property "Footprint" ""
-			(at 207.01 154.94 0)
-			(effects
-				(font
-					(size 1.27 1.27)
-				)
-			)
-			(hide yes)
-		)
-		(property "Datasheet" ""
-			(at 207.01 154.94 0)
-			(effects
-				(font
-					(size 1.27 1.27)
-				)
-			)
-			(hide yes)
+		(effects
+			(font (size 1.27 1.27))
+			(justify left)
 		)
-		(property "Description" ""
+		(property "Intersheetrefs" "${INTERSHEET_REFS}"
 			(at 207.01 154.94 0)
-			(effects
-				(font
-					(size 1.27 1.27)
-				)
-			)
-			(hide yes)
-		)
-		(pin "1"
-		)
-		(instances
-			(project "NeuralCard"
-				(path "/a1b2c3d4-0001-4000-8000-000000000001"
-					(reference "#PWR024")
-					(unit 1)
-				)
-			)
+			(effects (font (size 1.27 1.27)) (hide yes))
 		)
 	)
